File: SACRED_PCB/mqp2.kicad_sch (KiCad schematic)
At the start: 15 parts, among them U1 INA129, U2 Teensy4.1, U3 74VHC9164FT, U4 CD4066BE, U5 CD4066BE, U6 CD4066BE, U7 CD4066BE

Commit message: PCB schematic and a bunch of other stuff
Parts:
- added J1: Screw_Terminal_01x02, symbol Connector:Screw_Terminal_01x02
- added U8: CD74HC4067M, Package_SO:SOIC-24W_7.5x15.4mm_P1.27mm, symbol 74xx:CD74HC4067M
Connections:
- net VCC: no longer U2.46 (3V3)
- net at U1.6: no longer U2.36 (14_A0_TX3_SPDIF_OUT)
- net Earth: now reaches U2.1 (GND)
- net Earth: now also U2.34 (GND), U2.47 (GND), J1.2 (Pin_2)
- new net +12V: J1.1 (Pin_1)
- no-connect marks 0 -> 14
Other:
- note added: "12V Power in"
- note added: "Note: Be sure to cut the Vin-VUSB Jumper on the Teensy Power comes in from USB only"
- moved on the sheet: R1, R2, R3, RG, RV1, RV2, RV3, RV4, U1, U2, U3, U4A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
