File: SACRED_PCB/analog_channels.kicad_sch (KiCad schematic)
At the start: 19 parts, among them J14 Conn_01x16, J15 Screw_Terminal_01x04, J16 Screw_Terminal_01x02, U4 CD74HCT4067QM96Q, U7 OPA607Q1

Commit message: Proper arm generation and PCB progress
Parts:
- removed R2: 100k, symbol Device:R_Small_US
- removed R21: 3M, symbol Device:R_Small_US
- added JP3: Solder _Bridge, Jumper:SolderJumper-2_P1.3mm_Bridged_RoundedPad1.0x1.5mm, symbol Jumper:SolderJumper_2_Bridged
- added R2: R_Trim, OptoDevice:R_LDR_5.1x4.3mm_P3.4mm_Vertical, symbol Device:R_Trim
- added R6: 100k, Resistor_SMD:R_0805_2012Metric_Pad1.20x1.40mm_HandSolder, symbol Device:R_Small_US
- C10, C7, C8, C9: footprint (none) -> Capacitor_SMD:C_0805_2012Metric_Pad1.18x1.45mm_HandSolder
- C5: renamed from C11; footprint (none) -> Capacitor_SMD:C_0805_2012Metric_Pad1.18x1.45mm_HandSolder
- C6: renamed from C12; footprint (none) -> Capacitor_SMD:C_0805_2012Metric_Pad1.18x1.45mm_HandSolder
- J12: renamed from J15; footprint (none) -> TerminalBlock:TerminalBlock_MaiXu_MX126-5.0-05P_1x05_P5.00mm
- J13: renamed from J16; footprint (none) -> TerminalBlock_MetzConnect:TerminalBlock_MetzConnect_Type011_RT05502HBWC_1x02_P5.00mm_Horizontal
- J14: footprint (none) -> Connector_PinHeader_2.54mm:PinHeader_1x16_P2.54mm_Vertical
- JP1: renamed from JP3; footprint (none) -> Jumper:SolderJumper-2_P1.3mm_Bridged_RoundedPad1.0x1.5mm
- JP2: renamed from JP4; footprint (none) -> Jumper:SolderJumper-2_P1.3mm_Bridged_RoundedPad1.0x1.5mm
- R1, R3: footprint (none) -> Resistor_SMD:R_0805_2012Metric_Pad1.20x1.40mm_HandSolder
- R4, R5: footprint (none) -> Resistor_SMD:R_0805_2012Metric_Pad1.20x1.40mm_HandSolder; now not fitted
- renumbered U7 to U5
Connections:
- net +12V: now also J12.3 (Pin_3); no longer J12.1 (Pin_1)
- net +3.3V: now also J12.1 (Pin_1); no longer J12.3 (Pin_3)
- net AnalogX: now also JP3.1 (A), R6.1
- net at C9.1, U5.4 (-): now also R2.2
- new net: JP3.2 (B), R2.1, R6.2
Other:
- note added: "Emergency resistor to help the trim pot"
- moved on the sheet: C10, C8, C9, R3

Commit message: PCB Rev 0.1
Parts:
- removed C10: 100nF, Capacitor_SMD:C_0805_2012Metric_Pad1.18x1.45mm_HandSolder, symbol Device:C_Small
- removed J12: Screw_Terminal_01x04, TerminalBlock:TerminalBlock_MaiXu_MX126-5.0-05P_1x05_P5.00mm, symbol Connector:Screw_Terminal_01x04
- removed J14: Conn_01x16, Connector_PinHeader_2.54mm:PinHeader_1x16_P2.54mm_Vertical, symbol Connector_Generic:Conn_01x16
- added C3, C4: 10uF, Capacitor_SMD:C_1206_3216Metric, symbol Device:C_Small
- added J12: Screw_Terminal_01x04, TerminalBlock_Phoenix:TerminalBlock_Phoenix_MKDS-1,5-3-5.08_1x03_P5.08mm_Horizontal, symbol Connector:Screw_Terminal_01x03
- added J14, J18: Conn_01x16, Connector_PinHeader_2.54mm:PinHeader_1x08_P2.54mm_Vertical, symbol Connector_Generic:Conn_01x08
- added J17: Analog 0, Connector_PinHeader_2.54mm:PinHeader_1x05_P2.54mm_Vertical, symbol Connector_Generic:Conn_01x05
- added U2: AMS1117-3.3, Package_TO_SOT_SMD:SOT-223-3_TabPin2, symbol Regulator_Linear:AMS1117-3.3
- R2: footprint OptoDevice:R_LDR_5.1x4.3mm_P3.4mm_Vertical -> Potentiometer_THT:Potentiometer_Bourns_3296W_Vertical
Connections:
- net +12V: now also J12.2 (Pin_2)
- net +3.3V: now also C4.1, U2.2 (VO)
- net +5V: now also C3.1, J12.3 (Pin_3), U2.3 (VI)
- net AnalogX: now also J17.1 (Pin_1)
- net GND: now also C3.2, C4.2, J12.1 (Pin_1), U2.1 (GND)
- net MUX_0: now also J17.5 (Pin_5)
- net MUX_1: now also J17.4 (Pin_4)
- net MUX_2: now also J17.3 (Pin_3)
- net MUX_3: now also J17.2 (Pin_2)
- net at U4.9 (I0): now also J14.1 (Pin_1)
- net at U4.22 (I9): now also J18.2 (Pin_2)
- net at U4.21 (I10): now also J18.3 (Pin_3)
- net at U4.20 (I11): now also J18.4 (Pin_4)
- net at U4.19 (I12): now also J18.5 (Pin_5)
- net at U4.18 (I13): now also J18.6 (Pin_6)
- net at U4.17 (I14): now also J18.7 (Pin_7)
- net at U4.16 (I15): now also J18.8 (Pin_8)
- net at U4.8 (I1): now also J14.2 (Pin_2)
- net at U4.7 (I2): now also J14.3 (Pin_3)
- net at U4.6 (I3): now also J14.4 (Pin_4)
- net at U4.5 (I4): now also J14.5 (Pin_5)
- net at U4.4 (I5): now also J14.6 (Pin_6)
- net at U4.3 (I6): now also J14.7 (Pin_7)
- net at U4.2 (I7): now also J14.8 (Pin_8)
- net at U4.23 (I8): now also J18.1 (Pin_1)
Other:
- note added: "3.3V Regulator"

Commit message: PCB with rivets
Parts:
- R1, R3, R4, R5, R6: footprint Resistor_SMD:R_0805_2012Metric_Pad1.20x1.40mm_HandSolder -> Resistor_SMD:R_0603_1608Metric_Pad0.98x0.95mm_HandSolder
Changed lines of the file:
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@@
 			)
 		)
-		(property "Footprint" "Resistor_SMD:R_0805_2012Metric_Pad1.20x1.40mm_HandSolder"
+		(property "Footprint" "Resistor_SMD:R_0603_1608Metric_Pad0.98x0.95mm_HandSolder"
 			(at 120.65 101.6 0)
 			(effects
@@
 			)
 		)
-		(property "Footprint" "Resistor_SMD:R_0805_2012Metric_Pad1.20x1.40mm_HandSolder"
+		(property "Footprint" "Resistor_SMD:R_0603_1608Metric_Pad0.98x0.95mm_HandSolder"
 			(at 76.2 114.3 0)
 			(effects
@@
 			)
 		)
-		(property "Footprint" "Resistor_SMD:R_0805_2012Metric_Pad1.20x1.40mm_HandSolder"
+		(property "Footprint" "Resistor_SMD:R_0603_1608Metric_Pad0.98x0.95mm_HandSolder"
 			(at 120.65 130.81 0)
 			(effects
@@
 			)
 		)
-		(property "Footprint" "Resistor_SMD:R_0805_2012Metric_Pad1.20x1.40mm_HandSolder"
+		(property "Footprint" "Resistor_SMD:R_0603_1608Metric_Pad0.98x0.95mm_HandSolder"
 			(at 91.44 114.3 0)
 			(effects
@@
 			)
 		)
-		(property "Footprint" "Resistor_SMD:R_0805_2012Metric_Pad1.20x1.40mm_HandSolder"
+		(property "Footprint" "Resistor_SMD:R_0603_1608Metric_Pad0.98x0.95mm_HandSolder"
 			(at 120.65 115.57 0)
 			(effects
