File: Daughter_PCB/Daughter_PCB.kicad_sch (KiCad schematic)
At the start: 22 parts, among them J1 Screw_Terminal_01x02, J10 Conn_01x11, J11 Conn_01x13, J15 Screw_Terminal_01x04, J16 Conn_01x04, J2 Analog 0, J3 Analog 1, J4 Stepper 0, J5 Stepper 1, J6 Analog 2, J7 Stepper 2, J8 Stepper 3, J9 Analog 3, U1 AMS1117-5.0, U3 Teensy4.1

Commit message: Saving more
Parts:
- renumbered J11 to J10, J10 to J11, J16 to J12, J15 to J13, J7 to J5, J5 to J6, J8 to J7, J6 to J8, U3 to U2
Connections:
- net GND: no longer J10.4 (Pin_4), U2.34 (GND)
- net MUX_0: now also J2.3 (Pin_3), J3.3 (Pin_3), J8.3 (Pin_3), J9.3 (Pin_3), U2.40 (18_A4_SDA); no longer J2.2 (Pin_2), J3.2 (Pin_2), J8.2 (Pin_2), J9.2 (Pin_2), U2.41 (19_A5_SCL)
- net MUX_1: now also J2.2 (Pin_2), J3.2 (Pin_2), J8.2 (Pin_2), J9.2 (Pin_2), U2.41 (19_A5_SCL); no longer J2.3 (Pin_3), J3.3 (Pin_3), J8.3 (Pin_3), J9.3 (Pin_3), U2.40 (18_A4_SDA)
- new net Pin_GND: J10.4 (Pin_4), U2.34 (GND)
